Commit message: update readme

File: projects/quadruped_simulator/code/lib/URDF/05-sarge5_v1.urdf (robot description, URDF)
Before this commit: robot sarge5_v1, 17 links, 16 joints
Links:
- link back_left_foot: geometry collision mesh filename=../lib/STL/sarge5_foot.stl scale=0.01 0.01 0.01; visual mesh filename=../lib/STL/sarge5_foot.stl scale=0.01 0.01 0.01
- link back_left_hip: geometry collision mesh filename=../lib/STL/sarge5_hip.stl scale=0.01 0.01 0.01; visual mesh filename=../lib/STL/sarge5_hip.stl scale=0.01 0.01 0.01
- link back_left_knee: geometry collision mesh filename=../lib/STL/sarge5_knee.stl scale=0.01 0.01 0.01; visual mesh filename=../lib/STL/sarge5_knee.stl scale=0.01 0.01 0.01
- link back_right_foot: geometry collision mesh filename=../lib/STL/sarge5_foot.stl scale=0.01 0.01 0.01; visual mesh filename=../lib/STL/sarge5_foot.stl scale=0.01 0.01 0.01
- link back_right_hip: geometry collision mesh filename=../lib/STL/sarge5_hip.stl scale=0.01 0.01 0.01; visual mesh filename=../lib/STL/sarge5_hip.stl scale=0.01 0.01 0.01
- link back_right_knee: geometry collision mesh filename=../lib/STL/sarge5_knee.stl scale=0.01 0.01 0.01; visual mesh filename=../lib/STL/sarge5_knee.stl scale=0.01 0.01 0.01
- link base_link: geometry collision mesh filename=../lib/STL/sarge5_body_v2.stl scale=0.001 0.001 0.001; visual mesh filename=../lib/STL/sarge5_body_v2.stl scale=0.001 0.001 0.001
- link front_left_foot: geometry collision mesh filename=../lib/STL/sarge5_foot.stl scale=0.01 0.01 0.01; visual mesh filename=../lib/STL/sarge5_foot.stl scale=0.01 0.01 0.01
- link front_left_hip: geometry collision mesh filename=../lib/STL/sarge5_hip.stl scale=0.01 0.01 0.01; visual mesh filename=../lib/STL/sarge5_hip.stl scale=0.01 0.01 0.01
- link front_left_knee: geometry collision mesh filename=../lib/STL/sarge5_knee.stl scale=0.01 0.01 0.01; visual mesh filename=../lib/STL/sarge5_knee.stl scale=0.01 0.01 0.01
- link front_right_foot: geometry collision mesh filename=../lib/STL/sarge5_foot.stl scale=0.01 0.01 0.01; visual mesh filename=../lib/STL/sarge5_foot.stl scale=0.01 0.01 0.01
- link front_right_hip: geometry collision mesh filename=../lib/STL/sarge5_hip.stl scale=0.01 0.01 0.01; visual mesh filename=../lib/STL/sarge5_hip.stl scale=0.01 0.01 0.01
- link front_right_knee: geometry collision mesh filename=../lib/STL/sarge5_knee.stl scale=0.01 0.01 0.01; visual mesh filename=../lib/STL/sarge5_knee.stl scale=0.01 0.01 0.01

File: projects/quadruped_simulator/code/lib/URDF/05-sarge5_v1_stuck.urdf (robot description, URDF)
Before this commit: robot sarge5_v1, 18 links, 17 joints
Links:
- link back_left_foot: geometry collision mesh filename=../lib/STL/sarge5_foot.stl scale=0.01 0.01 0.01; visual mesh filename=../lib/STL/sarge5_foot.stl scale=0.01 0.01 0.01
- link back_left_hip: geometry collision mesh filename=../lib/STL/sarge5_hip.stl scale=0.01 0.01 0.01; visual mesh filename=../lib/STL/sarge5_hip.stl scale=0.01 0.01 0.01
- link back_left_knee: geometry collision mesh filename=../lib/STL/sarge5_knee.stl scale=0.01 0.01 0.01; visual mesh filename=../lib/STL/sarge5_knee.stl scale=0.01 0.01 0.01
- link back_right_foot: geometry collision mesh filename=../lib/STL/sarge5_foot.stl scale=0.01 0.01 0.01; visual mesh filename=../lib/STL/sarge5_foot.stl scale=0.01 0.01 0.01
- link back_right_hip: geometry collision mesh filename=../lib/STL/sarge5_hip.stl scale=0.01 0.01 0.01; visual mesh filename=../lib/STL/sarge5_hip.stl scale=0.01 0.01 0.01
- link back_right_knee: geometry collision mesh filename=../lib/STL/sarge5_knee.stl scale=0.01 0.01 0.01; visual mesh filename=../lib/STL/sarge5_knee.stl scale=0.01 0.01 0.01
- link base_link: geometry collision mesh filename=../lib/STL/sarge5_body_v2.stl scale=0.001 0.001 0.001; visual mesh filename=../lib/STL/sarge5_body_v2.stl scale=0.001 0.001 0.001
- link front_left_foot: geometry collision mesh filename=../lib/STL/sarge5_foot.stl scale=0.01 0.01 0.01; visual mesh filename=../lib/STL/sarge5_foot.stl scale=0.01 0.01 0.01
- link front_left_hip: geometry collision mesh filename=../lib/STL/sarge5_hip.stl scale=0.01 0.01 0.01; visual mesh filename=../lib/STL/sarge5_hip.stl scale=0.01 0.01 0.01
- link front_left_knee: geometry collision mesh filename=../lib/STL/sarge5_knee.stl scale=0.01 0.01 0.01; visual mesh filename=../lib/STL/sarge5_knee.stl scale=0.01 0.01 0.01
- link front_right_foot: geometry collision mesh filename=../lib/STL/sarge5_foot.stl scale=0.01 0.01 0.01; visual mesh filename=../lib/STL/sarge5_foot.stl scale=0.01 0.01 0.01
- link front_right_hip: geometry collision mesh filename=../lib/STL/sarge5_hip.stl scale=0.01 0.01 0.01; visual mesh filename=../lib/STL/sarge5_hip.stl scale=0.01 0.01 0.01
- link front_right_knee: geometry collision mesh filename=../lib/STL/sarge5_knee.stl scale=0.01 0.01 0.01; visual mesh filename=../lib/STL/sarge5_knee.stl scale=0.01 0.01 0.01
